File: Socket housing AWI (max6921)/proto.kicad_pcb (KiCad board)
At the start: 2 copper layers, 38.1 x 38.1 mm, 5 parts, among them P1 CONN_01X14, P2 CONN_01X14, P4 CONN_01X14, P5 CONN_01X14, U1 MAX6902

Commit message: Add files via upload
Parts:
- U1: footprint mod_reveil:MAX6921 - SOP28 -> MAX6921-SOP28
Routing:
- net Net-(P1-Pad14): track 18.6 -> 16.1 mm
- net Net-(P1-Pad3): track 14.1 -> 16.5 mm
- net Net-(P1-Pad2): track 15.4 -> 17.3 mm
- net Net-(P4-Pad14): track 12.6 -> 11.0 mm
- net Net-(P4-Pad12): track 16.1 -> 14.5 mm
- net Net-(P1-Pad13): track 16.8 -> 15.3 mm
- net Net-(P4-Pad13): track 16.5 -> 15.3 mm
- net Net-(P4-Pad11): track 15.1 -> 14.0 mm
- net Net-(P1-Pad10): track 13.0 -> 13.9 mm
- net Net-(P1-Pad5): track 13.0 -> 13.8 mm
- net Net-(P1-Pad12): track 15.2 -> 14.5 mm
Other:
- net class Default: clearance 0.4 -> 0.6
- rule trace_clearance: 0.4 -> 0.6
